File: HW #2/HW2/HW2_Schematics.brd (EAGLE design)
At the start: 160 x 100 mm, 23 parts, among them J1 USB-MB-H

Commit message: Board File Created
Parts:
- U$6, U$7: value CONN_010 -> CONN_015; device Honghe_Qi_ME433_HW2_Library:CONN_010 -> Honghe_Qi_ME433_HW2_Library:1X15
- moved U$2 68.3 mm to (-31.8, 20.3)
- moved U$1 64.4 mm to (-33.0, 7.62)
- moved U$9 37.6 mm to (-17.8, 61.0)
- moved C8 32.7 mm to (-16.5, 54.6)
- moved R3 30.9 mm to (-19.1, 64.8)
- moved LED2 28.4 mm to (-21.6, 71.1)
- moved C6 27.7 mm to (-21.6, 45.7)
- moved C5 12.7 mm to (-54.6, 47.0)
- moved U$3 12.7 mm to (-49.5, 66.0)
- moved C7 12.7 mm to (-34.3, 45.7)
- moved R4 12.7 mm to (-31.8, 64.8)
- moved C1 12.7 mm to (-41.9, 47.0)
- moved C4 12.7 mm to (-48.3, 47.0)
- moved LED1 11.4 mm to (-31.8, 71.1)
- moved R2 10.2 mm to (-47.0, 59.7)
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Connections:
- removed net RB10: U$1.8
- removed net RB11: U$1.9
- new net RC8: U$1.4, U$6.12
- new net RC9: U$1.5, U$6.11
- net +3V3: now also U$6.2
- net +5V: now also U$7.2
- net D+: now also U$1.8; no longer U$1.4
- net D-: now also U$1.9; no longer U$1.5
- net GND: now also U$6.1, U$7.1
- net RA0: now also U$6.5
- net RA1: now also U$6.4
- net RA10: now also U$6.9
- net RA4/LED: now also U$7.9
- net RA7: now also U$6.8
- net RA8: now also U$7.11
- net RA9: now also U$7.8
- net RB13: now also U$6.10
- net RB14: now also U$6.7
- net RB15: now also U$6.6
- net RB2: now also U$6.3
- net RB3: now also U$7.15
- net RB7: now also U$7.4
- net RB8: now also U$7.3
- net RB9: now also U$6.15
- net RC0: now also U$7.14
- net RC1: now also U$7.13
- net RC2: now also U$7.12
- net RC3: now also U$7.7
- net RC4: now also U$7.6
- net RC5: now also U$7.5
- net RC6: now also U$6.14
- net RC7: now also U$6.13
- net USER/RB4: now also U$7.10
