File: HW #2/HW2/HW2_Schematics.sch (EAGLE design)
At the start: 23 parts, among them J1 USB-MB-H

Commit message: Board File Created
Parts:
- U$6, U$7: value CONN_010 -> CONN_015; device Honghe_Qi_ME433_HW2_Library:CONN_010 -> Honghe_Qi_ME433_HW2_Library:CONN_015
Connections:
- net +3V3: now also U$6.2
- net +5V: now also U$7.2
- net GND: now also U$6.1, U$7.1
- net RA0: now also U$6.5
- net RA1: now also U$6.4
- net RA10: now also U$6.9
- net RA4/LED: now also U$7.9
- net RA7: now also U$6.8
- net RA8: now also U$7.11
- net RA9: now also U$7.8
- net RB13: now also U$6.10
- net RB14: now also U$6.7
- net RB15: now also U$6.6
- net RB2: now also U$6.3
- net RB3: now also U$7.15
- net RB7: now also U$7.4
- net RB8: now also U$7.3
- net RB9: now also U$6.15
- net RC0: now also U$7.14
- net RC1: now also U$7.13
- net RC2: now also U$7.12
- net RC3: now also U$7.7
- net RC4: now also U$7.6
- net RC5: now also U$7.5
- net RC6: now also U$6.14
- net RC7: now also U$6.13
- net RC8: now also U$6.12
- net RC9: now also U$6.11
- net USER/RB4: now also U$7.10
