File: HW #3/HW3_Board.brd (EAGLE design)
At the start: 100 x 100 mm, 23 parts, among them J1 USB-MB-H

Commit message: Board Created
Parts:
- moved U$4 91.9 mm to (25.4, 3.81), turned to 180 degrees
- moved R3 82.9 mm to (38.1, 3.81), turned to 180 degrees
- moved C8 3.81 mm to (49.5, 22.9)
- moved C3 2.54 mm to (49.5, 54.6)
- moved U$9 1.17 mm to (30.9, 37.6)
- moved J1 0.18 mm to (3.81, 83.7)
- flipped C4 to the top, turned to 270 degrees
Routing:
- net +3V3: track 0.00 -> 214.1 mm, vias 0 -> 6
- net +5V: track 0.00 -> 199.4 mm, vias 0 -> 2
- net RA4/LED: track 0.00 -> 109.9 mm, vias 0 -> 2
- net USER/RB4: track 0.00 -> 109.7 mm, vias 0 -> 2
- net D+: track 0.00 -> 82.4 mm, vias 0 -> 2
- net MCLR: track 0.00 -> 78.5 mm, vias 0 -> 2
- net D-: track 0.00 -> 77.6 mm, vias 0 -> 1
- net PGC: track 0.00 -> 63.9 mm, vias 0 -> 2
- net RB2: track 0.00 -> 62.7 mm, vias 0 -> 2
- net ID: track 0.00 -> 61.3 mm, vias 0 -> 2
- net PGD: track 0.00 -> 60.3 mm
- net RB8: track 0.00 -> 59.9 mm
- net RB7: track 0.00 -> 59.1 mm
- net RC5: track 0.00 -> 55.5 mm
- net RA1: track 0.00 -> 54.6 mm
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
Commit message: Board Finished
Parts:
- C3: value (none) -> 0.1uF
Connections:
- removed net N$5: C1.1, U$1.28
- net +3V3: now also C1.1, U$1.28
Routing:
- net +3V3: track 214.1 -> 228.3 mm
- net N$5: track 7.43 -> 0.00 mm
- net GND: track 11.3 -> 13.4 mm
- net N$1: vias 2 -> 1
Other:
- board text added: "+"
- board text added: "3V3"
- board text added: "5V"
- board text added: "A0"
- board text added: "A1"
- board text added: "A10"
- board text added: "A4"
- board text added: "A7"
- board text added: "A8"
- board text added: "A9"
- board text added: "B13"
- board text added: "B14"
- board text added: "B15"
- board text added: "B2"
- board text added: "B4"
- board text added: "B7"
- board text added: "B8"
- board text added: "B9"
- board text added: "C0"
- board text added: "C1"
- board text added: "C2"
- board text added: "C3"
- board text added: "C4"
- board text added: "C5"
- board text added: "C6"
- board text added: "C7"
- board text added: "C8"
- board text added: "C9"
- board text added: "GND"
- board text added: "HONGHE QI ME433 SPRING"

Commit message: Gerber File Created
Parts:
- moved C6 1.09 mm to (37.0, 36.9)
Routing:
- net +3V3: track 228.3 -> 226.6 mm
- net GND: track 13.4 -> 14.5 mm
- net N$4: track 9.01 -> 10.1 mm
Other:
- board text added: "10uF"
